Commit message: Update taweek9.urdf

File: gazebo_friction_test/urdf/taweek9.urdf (robot description, URDF)
Before this commit: robot urdf_test, 5 links, 4 joints
Links:
- link base_link: mass 5 -> None; geometry 
- link link_1: mass 1 -> None; geometry 
Joints:
- joint first_joint: origin xyz=0.5 1 0.7  rpy=0.7854 1.570796 0.7854 -> xyz=0 0 0.5  rpy=0 0 0
- joint second_joint: axis 0 0 1 -> 0 1 0; origin xyz=0.5 0.3 0.1  rpy=0 1.5707963 0 -> xyz=0 0 0.1  rpy=0 0 0
- joint third_joint: axis 0 1 0 -> 1 0 0
