Commit message: cartpole updated

File: cartpole_control/urdf/cartpole_v1.urdf (robot description, URDF)
Before this commit: robot cartpole, 4 links, 3 joints
Links:
- link cart: geometry collision mesh filename=package://cartpole_control/meshes/cart.stl; visual mesh filename=package://cartpole_control/meshes/cart.stl
- link pole: geometry collision mesh filename=package://cartpole_control/meshes/pole.stl; visual mesh filename=package://cartpole_control/meshes/pole.stl
- link stand: geometry collision mesh filename=package://cartpole_control/meshes/stand.stl; visual mesh filename=package://cartpole_control/meshes/stand.stl
